File: alpha-curISO.kicad_pcb (KiCad board)
At the start: 2 copper layers, 248.6 x 81.9 mm, 175 parts, among them SW1 SW_Push_45deg, SW10 SW_Push_45deg, SW11 SW_Push_45deg, SW12 SW_Push_45deg, SW12(2)1 SW_Push_45deg, SW13 SW_Push_45deg, SW14 SW_Push_45deg, SW15 SW_Push_45deg, SW16 SW_Push_45deg, SW17 SW_Push_45deg, SW18 SW_Push_45deg, SW19 SW_Push_45deg, SW2 SW_Push_45deg, SW20 SW_Push_45deg, SW21 SW_Push_45deg, SW22 SW_Push_45deg, SW23 SW_Push_45deg, SW24 SW_Push_45deg, SW24(1.5)1 SW_Push_45deg, SW25 SW_Push_45deg, SW25(1.5)1 SW_Push_45deg, SW26 SW_Push_45deg, SW26(2)1 SW_Push_45deg, SW26(ISO)1 SW_Push_45deg, SW27(1.25)1 SW_Push_45deg, SW27(1.5)1 SW_Push_45deg, SW27(ortho)1 SW_Push_45deg, SW28 SW_Push_45deg, SW28(1.5stagger)1 SW_Push_45deg, SW28(ortho)1 SW_Push_45deg, SW29 SW_Push_45deg, SW29(1.5stagger)1 SW_Push_45deg, SW29(ortho)1 SW_Push_45deg, SW3 SW_Push_45deg, SW30 SW_Push_45deg, SW30(1.5stagger)1 SW_Push_45deg, SW30(ortho)1 SW_Push_45deg, SW31 SW_Push_45deg, SW31(1.5stagger)1 SW_Push_45deg, SW31(ortho)1 SW_Push_45deg, SW32 SW_Push_45deg, SW32(1.5stagger)1 SW_Push_45deg, SW32(ortho)1 SW_Push_45deg, SW33 SW_Push_45deg, SW33(1.5stagger)1 SW_Push_45deg, SW33(ortho)1 SW_Push_45deg, SW34 SW_Push_45deg, SW34(1.5stagger)1 SW_Push_45deg, SW34(ortho)1 SW_Push_45deg, SW35 SW_Push_45deg, SW35(1.5stagger)1 SW_Push_45deg, SW35(ortho)1 SW_Push_45deg, SW36 SW_Push_45deg, SW36(1.5stagger)1 SW_Push_45deg, SW36(ortho)1 SW_Push_45deg, SW37 SW_Push_45deg, SW37(1.5stagger)1 SW_Push_45deg, SW37(ortho)1 SW_Push_45deg, SW38(1.25)1 SW_Push_45deg, SW38(1.5)1 SW_Push_45deg, SW38(ortho)1 SW_Push_45deg, SW39 SW_Push_45deg, SW39(1.5)1 SW_Push_45deg, SW4 SW_Push_45deg, SW40 SW_Push_45deg, SW40(3)1 SW_Push_45deg, SW41 SW_Push_45deg, SW41(1.5)1 SW_Push_45deg, SW42(1.25)1 SW_Push_45deg, SW42(1.5)1 SW_Push_45deg, SW42(3)1 SW_Push_45deg, SW43(1.75)1 SW_Push_45deg, SW43(2)1 SW_Push_45deg, SW44(3)1 SW_Push_45deg, SW44(6)1 SW_Push_45deg, SW45(1.75)1 SW_Push_45deg, SW45(2)1 SW_Push_45deg, SW46(1.25)1 SW_Push_45deg, SW46(1.5)1 SW_Push_45deg, SW46(3)1 SW_Push_45deg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

Commit message: footprint WIP
Parts:
- moved SW24(1.5)1 394.4 mm to (230.2, 41.3)
- moved SW44(6)1 360.3 mm to (149.2, 134.1)
- moved SW26 331.1 mm to (261.1, 79.4)
- moved SW38(1.25)1 322.6 mm to (258.8, 98.4)
- moved SW10 298.7 mm to (204.0, 60.3)
- moved SW38(ortho)1 293.6 mm to (261.1, 98.4)
- moved SW23 283.3 mm to (204.0, 79.4)
- moved SW13 275.3 mm to (261.1, 60.3)
- moved SW37(ortho)1 263.1 mm to (242.1, 98.4)
- moved SW36(ortho)1 262.5 mm to (223.0, 98.4)
- moved SW36 258.7 mm to (218.3, 98.4)
- moved SW11 250.5 mm to (223.0, 60.3)
- moved SW21 248.2 mm to (165.9, 79.4)
- moved SW19 247.6 mm to (127.8, 79.4)
- moved SW37 244.5 mm to (237.3, 98.4)
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