File: alpha-curISO.kicad_pcb (KiCad board)
At the start: 2 copper layers, 248.6 x 81.9 mm, 0 parts

Commit message: edited schematics, assigned footprints
4u spacebar missing, no appropriate footprint in library yet
Parts:
- added C1: 4.7uF, Capacitor_SMD:C_0805_2012Metric, F.Cu at (-152.4, 101.6)
- added C10: 22p, Capacitor_SMD:C_0805_2012Metric, F.Cu at (-152.4, 104.6)
- added C2: 2.2uF, Capacitor_SMD:C_0805_2012Metric_Pad1.18x1.45mm_HandSolder, F.Cu at (-141.1, 90.4)
- added C3: 1uf, Capacitor_SMD:C_0805_2012Metric, F.Cu at (191.9, -113.1)
- added C4: 10uF, Capacitor_SMD:C_0805_2012Metric, F.Cu at (-143.5, 93.4)
- added C5: 0.1uf, Capacitor_SMD:C_0805_2012Metric, F.Cu at (-143.5, 101.6)
- added C6: 0.1uf, Capacitor_SMD:C_0805_2012Metric, F.Cu at (-159.1, 107.6)
- added C7: 0.1uf, Capacitor_SMD:C_0805_2012Metric, F.Cu at (-147.9, 101.6)
- added C8: 0.1uf, Capacitor_SMD:C_0805_2012Metric, F.Cu at (-154.6, 107.6)
- added C9: 22p, Capacitor_SMD:C_0805_2012Metric, F.Cu at (-147.9, 104.6)
- added D1: D_Small, Diode_SMD:D_SOD-123F, F.Cu at (-97.5, 72.1)
- added D10: D_Small, Diode_SMD:D_SOD-123F, F.Cu at (-102.9, 72.1)
- added D11: D_Small, Diode_SMD:D_SOD-123F, F.Cu at (-157.7, 74.3)
- added D12: D_Small, Diode_SMD:D_SOD-123F, F.Cu at (-108.4, 75.4)
- added D13: D_Small, Diode_SMD:D_SOD-123F, F.Cu at (-152.3, 70.9)
- added D14: D_Small, Diode_SMD:D_SOD-123F, F.Cu at (-102.9, 75.4)
- added D15: D_Small, Diode_SMD:D_SOD-123F, F.Cu at (-97.5, 78.8)
- added D16: D_Small, Diode_SMD:D_SOD-123F, F.Cu at (-113.9, 78.8)
- added D17: D_Small, Diode_SMD:D_SOD-123F, F.Cu at (-102.9, 78.8)
- added D18: D_Small, Diode_SMD:D_SOD-123F, F.Cu at (-135.8, 78.8)
- added D19: D_Small, Diode_SMD:D_SOD-123F, F.Cu at (-130.3, 82.1)
- added D2: D_Small, Diode_SMD:D_SOD-123F, F.Cu at (-113.9, 72.1)
- added D20: D_Small, Diode_SMD:D_SOD-123F, F.Cu at (-135.8, 75.4)
- added D21: D_Small, Diode_SMD:D_SOD-123F, F.Cu at (-108.4, 78.8)
- added D22: D_Small, Diode_SMD:D_SOD-123F, F.Cu at (-130.3, 72.1)
- added D23: D_Small, Diode_SMD:D_SOD-123F, F.Cu at (-157.7, 70.9)
- added D24: D_Small, Diode_SMD:D_SOD-123F, F.Cu at (-113.9, 75.4)
- added D25: D_Small, Diode_SMD:D_SOD-123F, F.Cu at (-157.7, 81.0)
- added D26: D_Small, Diode_SMD:D_SOD-123F, F.Cu at (-92.0, 72.1)
- added D27: D_Small, Diode_SMD:D_SOD-123F, F.Cu at (-119.4, 75.4)
- added D28: D_Small, Diode_SMD:D_SOD-123F, F.Cu at (-146.8, 82.1)
- added D29: D_Small, Diode_SMD:D_SOD-123F, F.Cu at (-146.8, 78.8)
- added D3: D_Small, Diode_SMD:D_SOD-123F, F.Cu at (-108.4, 82.1)
- added D30: D_Small, Diode_SMD:D_SOD-123F, F.Cu at (-157.7, 77.6)
- added D31: D_Small, Diode_SMD:D_SOD-123F, F.Cu at (-108.4, 72.1)
- added D32: D_Small, Diode_SMD:D_SOD-123F, F.Cu at (-141.3, 75.4)
- added D33: D_Small, Diode_SMD:D_SOD-123F, F.Cu at (-135.8, 82.1)
- added D34: D_Small, Diode_SMD:D_SOD-123F, F.Cu at (-119.4, 78.8)
- added D35: D_Small, Diode_SMD:D_SOD-123F, F.Cu at (-141.3, 78.8)
- added D36: D_Small, Diode_SMD:D_SOD-123F, F.Cu at (-130.3, 75.4)
- added D37: D_Small, Diode_SMD:D_SOD-123F, F.Cu at (-124.9, 78.8)
- added D38: D_Small, Diode_SMD:D_SOD-123F, F.Cu at (-130.3, 78.8)
- added D39: D_Small, Diode_SMD:D_SOD-123F, F.Cu at (-124.9, 72.1)
- added D4: D_Small, Diode_SMD:D_SOD-123F, F.Cu at (-146.8, 72.1)
- added D40: D_Small, Diode_SMD:D_SOD-123F, F.Cu at (-152.3, 81.0)
- added D41: D_Small, Diode_SMD:D_SOD-123F, F.Cu at (-135.8, 72.1)
- added D42: D_Small, Diode_SMD:D_SOD-123F, F.Cu at (-124.9, 82.1)
- added D43: D_Small, Diode_SMD:D_SOD-123F, F.Cu at (-102.9, 82.1)
- added D44: D_Small, Diode_SMD:D_SOD-123F, F.Cu at (-119.4, 72.1)
- added D45: D_Small, Diode_SMD:D_SOD-123F, F.Cu at (-113.9, 82.1)
- added D46: D_Small, Diode_SMD:D_SOD-123F, F.Cu at (-124.9, 75.4)
- added D47: D_Small, Diode_SMD:D_SOD-123F, F.Cu at (-97.5, 75.4)
- added D48: D_Small, Diode_SMD:D_SOD-123F, F.Cu at (-141.3, 72.1)
- added D49: D_Small, Diode_SMD:D_SOD-123F, F.Cu at (-152.3, 77.6)
- added D5: D_Small, Diode_SMD:D_SOD-123F, F.Cu at (-152.3, 74.3)
- added D6: D_Small, Diode_SMD:D_SOD-123F, F.Cu at (-119.4, 82.1)
- added D7: D_Small, Diode_SMD:D_SOD-123F, F.Cu at (-92.0, 75.4)
- added D8: D_Small, Diode_SMD:D_SOD-123F, F.Cu at (-141.3, 82.1)
- added D9: D_Small, Diode_SMD:D_SOD-123F, F.Cu at (-146.8, 75.4)
- added F1: Polyfuse_Small, Fuse:Fuse_1206_3216Metric_Pad1.42x1.75mm_HandSolder, F.Cu at (-151.7, 97.3)
- added OL1: OLED, kbd:OLED_v2, F.Cu at (-172.5, 126.2)
- added R1: 10k, Resistor_SMD:R_0805_2012Metric, F.Cu at (-159.3, 110.6)
- added R2: 10k, Resistor_SMD:R_0805_2012Metric, F.Cu at (191.9, -107.2)
- added SW1: SW_Push_45deg, MX_Only:MXOnly-1U-NoLED, F.Cu at (59.5, -104.5)
- added SW10: SW_Push_45deg, MX_Only:MXOnly-1U-NoLED, F.Cu at (-94.1, 40.1)
- added SW11: SW_Push_45deg, MX_Only:MXOnly-1U-NoLED, F.Cu at (-23.9, 18.6)
- added SW12: SW_Push_45deg, MX_Only:MXOnly-1U-NoLED, F.Cu at (115.3, -84.3)
- added SW12(2)1: SW_Push_45deg, MX_Only:MXOnly-2U-NoLED, F.Cu at (-120.2, -42.0)
- added SW13: SW_Push_45deg, MX_Only:MXOnly-1U-NoLED, F.Cu at (-13.3, 38.8)
- added SW14: SW_Push_45deg, MX_Only:MXOnly-1U-NoLED, F.Cu at (95.1, -84.3)
- added SW15: SW_Push_45deg, MX_Only:MXOnly-1U-NoLED, F.Cu at (-73.9, 40.1)
- added SW16: SW_Push_45deg, MX_Only:MXOnly-1U-NoLED, F.Cu at (160.5, -104.5)
- added SW17: SW_Push_45deg, MX_Only:MXOnly-1U-NoLED, F.Cu at (40.3, -23.7)
- added SW18: SW_Push_45deg, MX_Only:MXOnly-1U-NoLED, F.Cu at (-20.3, -23.1)
- added SW19: SW_Push_45deg, MX_Only:MXOnly-1U-NoLED, F.Cu at (-119.0, 60.3)
- added SW2: SW_Push_45deg, MX_Only:MXOnly-1U-NoLED, F.Cu at (6.93, 37.5)
- added SW20: SW_Push_45deg, MX_Only:MXOnly-1U-NoLED, F.Cu at (79.7, -104.5)
- added SW21: SW_Push_45deg, MX_Only:MXOnly-1U-NoLED, F.Cu at (-60.7, -21.8)
- added SW22: SW_Push_45deg, MX_Only:MXOnly-1U-NoLED, F.Cu at (22.5, -64.1)
- added SW23: SW_Push_45deg, MX_Only:MXOnly-1U-NoLED, F.Cu at (-78.6, 60.3)
- added SW24: SW_Push_45deg, MX_Only:MXOnly-1U-NoLED, F.Cu at (135.5, -84.3)
- added SW24(1.5)1: SW_Push_45deg, MX_Only:MXOnly-1.5U-NoLED, F.Cu at (-164.2, 38.9)
- added SW25: SW_Push_45deg, MX_Only:MXOnly-1U-NoLED, F.Cu at (26.0, -3.50)
- added SW25(1.5)1: SW_Push_45deg, MX_Only:MXOnly-1.5U-NoLED, F.Cu at (-85.7, -21.8)
- added SW26: SW_Push_45deg, MX_Only:MXOnly-1U-NoLED, F.Cu at (-64.3, 18.6)
- added SW26(2)1: SW_Push_45deg, MX_Only:MXOnly-2U-NoLED, F.Cu at (-120.2, -21.1)
- added SW26(ISO)1: SW_Push_45deg, MX_Only:MXOnly-ISO-NoLED, F.Cu at (-161.8, 9.22)
- added SW27(1.25)1: SW_Push_45deg, MX_Only:MXOnly-1.25U-NoLED, F.Cu at (-20.2, -83.7)
- added SW27(1.5)1: SW_Push_45deg, MX_Only:MXOnly-1.5U-NoLED, F.Cu at (-164.2, 59.1)
- added SW27(ortho)1: SW_Push_45deg, MX_Only:MXOnly-1U-NoLED, F.Cu at (2.33, -64.1)
- added SW28: SW_Push_45deg, MX_Only:MXOnly-1U-NoLED, F.Cu at (-114.3, 40.1)
- added SW28(1.5stagger)1: SW_Push_45deg, MX_Only:MXOnly-1U-NoLED, F.Cu at (-34.6, -1.58)
- added SW28(ortho)1: SW_Push_45deg, MX_Only:MXOnly-1U-NoLED, F.Cu at (140.3, -104.5)
- added SW29: SW_Push_45deg, MX_Only:MXOnly-1U-NoLED, F.Cu at (29.6, -43.9)
- added SW29(1.5stagger)1: SW_Push_45deg, MX_Only:MXOnly-1U-NoLED, F.Cu at (-44.1, 18.6)
- added SW29(ortho)1: SW_Push_45deg, MX_Only:MXOnly-1U-NoLED, F.Cu at (123.5, -64.1)
- added SW3: SW_Push_45deg, MX_Only:MXOnly-1U-NoLED, F.Cu at (54.7, -84.3)
- added SW30: SW_Push_45deg, MX_Only:MXOnly-1U-NoLED, F.Cu at (70.0, -43.9)
- added SW30(1.5stagger)1: SW_Push_45deg, MX_Only:MXOnly-1U-NoLED, F.Cu at (62.9, -64.1)
- added SW30(ortho)1: SW_Push_45deg, MX_Only:MXOnly-1U-NoLED, F.Cu at (-75.0, -1.58)
- added SW31: SW_Push_45deg, MX_Only:MXOnly-1U-NoLED, F.Cu at (5.78, -2.87)
- added SW31(1.5stagger)1: SW_Push_45deg, MX_Only:MXOnly-1U-NoLED, F.Cu at (120.1, -104.5)
- added SW31(ortho)1: SW_Push_45deg, MX_Only:MXOnly-1U-NoLED, F.Cu at (2.17, 59.0)
- added SW32: SW_Push_45deg, MX_Only:MXOnly-1U-NoLED, F.Cu at (99.9, -104.5)
- added SW32(1.5stagger)1: SW_Push_45deg, MX_Only:MXOnly-1U-NoLED, F.Cu at (-10.8, -43.3)
- added SW32(ortho)1: SW_Push_45deg, MX_Only:MXOnly-1U-NoLED, F.Cu at (90.2, -43.9)
- added SW33: SW_Push_45deg, MX_Only:MXOnly-1U-NoLED, F.Cu at (-3.75, 17.3)
- added SW33(1.5stagger)1: SW_Push_45deg, MX_Only:MXOnly-1U-NoLED, F.Cu at (-54.8, -1.58)
- added SW33(ortho)1: SW_Push_45deg, MX_Only:MXOnly-1U-NoLED, F.Cu at (-58.4, 60.3)
- added SW34: SW_Push_45deg, MX_Only:MXOnly-1U-NoLED, F.Cu at (20.1, -23.7)
- added SW34(1.5stagger)1: SW_Push_45deg, MX_Only:MXOnly-1U-NoLED, F.Cu at (80.7, -23.7)
- added SW34(ortho)1: SW_Push_45deg, MX_Only:MXOnly-1U-NoLED, F.Cu at (16.5, 17.3)
- added SW35: SW_Push_45deg, MX_Only:MXOnly-1U-NoLED, F.Cu at (42.7, -64.1)
- added SW35(1.5stagger)1: SW_Push_45deg, MX_Only:MXOnly-1U-NoLED, F.Cu at (-53.7, 38.8)
- added SW35(ortho)1: SW_Push_45deg, MX_Only:MXOnly-1U-NoLED, F.Cu at (60.5, -23.7)
- added SW36: SW_Push_45deg, MX_Only:MXOnly-1U-NoLED, F.Cu at (-33.5, 38.8)
- added SW36(1.5stagger)1: SW_Push_45deg, MX_Only:MXOnly-1U-NoLED, F.Cu at (39.3, -104.5)
- added SW36(ortho)1: SW_Push_45deg, MX_Only:MXOnly-1U-NoLED, F.Cu at (34.5, -84.3)
- added SW37: SW_Push_45deg, MX_Only:MXOnly-1U-NoLED, F.Cu at (74.9, -84.3)
- added SW37(1.5stagger)1: SW_Push_45deg, MX_Only:MXOnly-1U-NoLED, F.Cu at (-84.5, 19.9)
- added SW37(ortho)1: SW_Push_45deg, MX_Only:MXOnly-1U-NoLED, F.Cu at (-18.0, 59.0)
- added SW38(1.25)1: SW_Push_45deg, MX_Only:MXOnly-1.25U-NoLED, F.Cu at (-20.2, -63.5)
- added SW38(1.5)1: SW_Push_45deg, MX_Only:MXOnly-1.5U-NoLED, F.Cu at (-47.6, -83.7)
- added SW38(ortho)1: SW_Push_45deg, MX_Only:MXOnly-1U-NoLED, F.Cu at (-14.4, -2.87)
- added SW39: SW_Push_45deg, MX_Only:MXOnly-1U-NoLED, F.Cu at (103.3, -64.1)
- added SW39(1.5)1: SW_Push_45deg, MX_Only:MXOnly-1.5U-NoLED, F.Cu at (-85.7, -42.0)
- added SW4: SW_Push_45deg, MX_Only:MXOnly-1U-NoLED, F.Cu at (-0.12, -23.1)
- added SW40: SW_Push_45deg, MX_Only:MXOnly-1U-NoLED, F.Cu at (46.2, -3.50)
- added SW40(3)1: SW_Push_45deg, MX_Only:MXOnly-3U-ReversedStabilizers-NoLED, F.Cu at (-149.9, -83.0)
- added SW41: SW_Push_45deg, MX_Only:MXOnly-1U-NoLED, F.Cu at (-139.2, 60.3)
- added SW41(1.5)1: SW_Push_45deg, MX_Only:MXOnly-1.5U-NoLED, F.Cu at (9.57, -84.3)
- added SW42(1.25)1: SW_Push_45deg, MX_Only:MXOnly-1.25U-NoLED, F.Cu at (-136.8, 40.1)
- added SW42(1.5)1: SW_Push_45deg, MX_Only:MXOnly-1.5U-NoLED, F.Cu at (-47.6, -63.5)
- added SW42(3)1: SW_Push_45deg, MX_Only:MXOnly-3U-ReversedStabilizers-NoLED, F.Cu at (-91.6, -83.0)
- added SW43(1.75)1: SW_Push_45deg, MX_Only:MXOnly-1.75U-NoLED, F.Cu at (11.9, -104.5)
- added SW43(2)1: SW_Push_45deg, MX_Only:MXOnly-2U-ReversedStabilizers-NoLED, F.Cu at (-159.4, -41.3)
- added SW44(3)1: SW_Push_45deg, MX_Only:MXOnly-3U-ReversedStabilizers-NoLED, F.Cu at (-91.6, -62.2)
- added SW44(6)1: SW_Push_45deg, MX_Only:MXOnly-6U-Centered-ReversedStabilizers-NoLED, F.Cu at (-121.3, -103.9)
- added SW45(1.75)1: SW_Push_45deg, MX_Only:MXOnly-1.75U-NoLED, F.Cu at (-132.1, -0.30)
- added SW45(2)1: SW_Push_45deg, MX_Only:MXOnly-2U-ReversedStabilizers-NoLED, F.Cu at (-159.4, -20.5)
- added SW46(1.25)1: SW_Push_45deg, MX_Only:MXOnly-1.25U-NoLED, F.Cu at (-107.1, 19.9)
- added SW46(1.5)1: SW_Push_45deg, MX_Only:MXOnly-1.5U-NoLED, F.Cu at (-100.0, -0.30)
- added SW46(3)1: SW_Push_45deg, MX_Only:MXOnly-3U-ReversedStabilizers-NoLED, F.Cu at (-34.4, -103.9)
- added SW47: SW_Push_45deg, MX_Only:MXOnly-1U-NoLED, F.Cu at (83.1, -64.1)
- added SW47(1.5)1: SW_Push_45deg, MX_Only:MXOnly-1.5U-NoLED, F.Cu at (-134.5, 19.9)
- added SW48: SW_Push_45deg, MX_Only:MXOnly-1U-NoLED, F.Cu at (-98.8, 60.3)
- added SW48(3)1: SW_Push_45deg, MX_Only:MXOnly-3U-ReversedStabilizers-NoLED, F.Cu at (-149.9, -62.2)
- added SW49: SW_Push_45deg, MX_Only:MXOnly-1U-NoLED, F.Cu at (49.8, -43.9)
- added SW49(1.5)1: SW_Push_45deg, MX_Only:MXOnly-1.5U-NoLED, F.Cu at (-56.0, -42.0)
- added SW5: SW_Push_45deg, MX_Only:MXOnly-1U-NoLED, F.Cu at (-38.2, 59.0)
- added SW6: SW_Push_45deg, MX_Only:MXOnly-1U-NoLED, F.Cu at (-31.0, -43.3)
- added SW7: SW_Push_45deg, MX_Only:MXOnly-1U-NoLED, F.Cu at (-40.5, -21.8)
- added SW8: SW_Push_45deg, MX_Only:MXOnly-1U-NoLED, F.Cu at (9.39, -43.9)
- added SW9: SW_Push_45deg, MX_Only:MXOnly-1U-NoLED, F.Cu at (36.7, 16.7)
- added SW_Push1: SW_PUSH, Button_Switch_SMD:SW_SPST_SKQG_WithoutStem, F.Cu at (-174.3, 131.4)
- added SW_Push2: SW_PUSH, Connector_PinHeader_2.54mm:PinHeader_1x02_P2.54mm_Vertical, F.Cu at (-163.6, 101.9)
- added SW_Push3: SW_PUSH, Button_Switch_SMD:SW_SPST_SKQG_WithoutStem, F.Cu at (-150.5, 92.3)
- added SW_rotary1: RotaryEncoder_Switch, Keebio-Parts:RotaryEncoder_EC11-no-legs, F.Cu at (-169.5, 76.9)
- added TP1: TPGND, TestPoint:TestPoint_THTPad_1.0x1.0mm_Drill0.5mm, F.Cu at (-164.4, 116.7)
- added TP2: TPVCC, TestPoint:TestPoint_THTPad_1.0x1.0mm_Drill0.5mm, F.Cu at (-161.3, 113.6)
- added TP3: TPCLK, TestPoint:TestPoint_THTPad_1.0x1.0mm_Drill0.5mm, F.Cu at (-164.4, 113.6)
- added TP4: TPDATA, TestPoint:TestPoint_THTPad_1.0x1.0mm_Drill0.5mm, F.Cu at (-158.3, 113.6)
- added TP5: TPRST, TestPoint:TestPoint_THTPad_1.0x1.0mm_Drill0.5mm, F.Cu at (-155.2, 113.6)
- added U1: SRV05-4, Package_TO_SOT_SMD:SOT-23-6, F.Cu at (-146.1, 97.9)
- added U2: ATmega32U4-M, Package_DFN_QFN:QFN-44-1EP_7x7mm_P0.5mm_EP5.2x5.2mm_ThermalVias, F.Cu at (185.1, -110.0)
- added UR1: 22, Resistor_SMD:R_0805_2012Metric, F.Cu at (196.4, -113.1)
- added UR2: 22, Resistor_SMD:R_0805_2012Metric, F.Cu at (191.9, -110.1)
- added UR3: 1M, Resistor_SMD:R_0805_2012Metric, F.Cu at (-163.7, 110.6)
- added UR4: 5.1k, Resistor_SMD:R_0805_2012Metric, F.Cu at (-154.9, 110.6)
- added UR5: 5.1k, Resistor_SMD:R_0805_2012Metric, F.Cu at (-150.2, 107.6)
- added UR6: 100k, Resistor_SMD:R_0805_2012Metric_Pad1.20x1.40mm_HandSolder, F.Cu at (-136.3, 93.3)
- added UR7: 4.7k, Resistor_SMD:R_0805_2012Metric_Pad1.20x1.40mm_HandSolder, F.Cu at (-136.3, 90.4)
- added UR8: 4.7k, Resistor_SMD:R_0805_2012Metric_Pad1.20x1.40mm_HandSolder, F.Cu at (-131.6, 90.4)
- added USB1: HRO-TYPE-C-31-M-12, Type-C:HRO-TYPE-C-31-M-12-HandSoldering, F.Cu at (-160.6, 98.8)
- added X1: Crystal_GND24_Small, Crystal:Crystal_SMD_3225-4Pin_3.2x2.5mm_HandSoldering, F.Cu at (-157.9, 102.4)

Commit message: arrange footprints
Parts:
- added SW_rotary2: RotaryEncoder_Switch, Keebio-Parts:RotaryEncoder_EC11-no-legs, F.Cu at (261.9, 58.7)
- added SW_rotary3: RotaryEncoder_Switch, Keebio-Parts:RotaryEncoder_EC11-no-legs, F.Cu at (147.6, 58.7)
- added SW_rotary4: RotaryEncoder_Switch, Keebio-Parts:RotaryEncoder_EC11-no-legs, F.Cu at (147.6, 77.8)
- added SW_rotary5: RotaryEncoder_Switch, Keebio-Parts:RotaryEncoder_EC11-no-legs, F.Cu at (100.0, 120.7)
- added SW_rotary6: RotaryEncoder_Switch, Keebio-Parts:RotaryEncoder_EC11-no-legs, F.Cu at (195.3, 120.7)
- C1, C10, C2, C3, C4, C5, C6, C7, C8, C9, D1, D10, D11, D12, D13, D14, D15, D16, D17, D18, D19, D2, D20, D21, D22, D23, D24, D25, D26, D27, D28, D29, D3, D30, D31, D32, D33, D34, D35, D36, D37, D38, D39, D4, D40, D41, D42, D43, D44, D45, D46, D47, D48, D49, D5, D6, D7, D8, D9, F1, R1, R2, SW_Push1, SW_Push3, TP1, TP2, TP3, TP4, TP5, U1, U2, UR1, UR2, UR3, UR4, UR5, UR6, UR7, UR8, USB1, X1: moved to B.Cu
- moved SW26(ISO)1 428.5 mm to (259.6, 87.3)
- moved SW48(3)1 426.9 mm to (238.1, 115.9)
- moved SW24(1.5)1 394.7 mm to (228.6, 77.8)
- moved SW12(2)1 386.0 mm to (252.4, 58.7)
- moved SW26(2)1 385.5 mm to (252.4, 77.8)
- moved SW47(1.5)1 370.9 mm to (223.8, 115.9)
- moved SW25(1.5)1 357.0 mm to (257.2, 77.8)
- moved SW45(2)1 355.3 mm to (166.7, 120.7)
- moved SW38(1.5)1 354.2 mm to (257.2, 96.8)
- moved SW44(6)1 350.3 mm to (147.6, 120.7)
- moved SW49(1.5)1 346.4 mm to (252.4, 115.9)
- moved SW48 341.5 mm to (238.1, 115.9)
- moved SW26 331.6 mm to (261.9, 77.8)
- moved SW43(2)1 330.4 mm to (128.6, 120.7)
- moved SW37(1.5stagger)1 327.1 mm to (233.4, 96.8)
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Other:
- board text added: "1 rotary"
- board text added: "2 rotaries"
- board text added: "EDGE CUT NEEDS TO BE ALIGNED TO FOOTPRINTS STILL"
- board text added: "indicator leds"
