File: alpha-curISO.kicad_pcb (KiCad board)
At the start: 2 copper layers, 248.6 x 81.9 mm, 175 parts, among them SW1 SW_Push_45deg, SW10 SW_Push_45deg, SW11 SW_Push_45deg, SW12 SW_Push_45deg, SW12(2)1 SW_Push_45deg, SW13 SW_Push_45deg, SW14 SW_Push_45deg, SW15 SW_Push_45deg, SW16 SW_Push_45deg, SW17 SW_Push_45deg, SW18 SW_Push_45deg, SW19 SW_Push_45deg, SW2 SW_Push_45deg, SW20 SW_Push_45deg, SW21 SW_Push_45deg, SW22 SW_Push_45deg, SW23 SW_Push_45deg, SW24 SW_Push_45deg, SW24(1.5)1 SW_Push_45deg, SW25 SW_Push_45deg, SW25(1.5)1 SW_Push_45deg, SW26 SW_Push_45deg, SW26(2)1 SW_Push_45deg, SW26(ISO)1 SW_Push_45deg, SW27(1.25)1 SW_Push_45deg, SW27(1.5)1 SW_Push_45deg, SW27(ortho)1 SW_Push_45deg, SW28 SW_Push_45deg, SW28(1.5stagger)1 SW_Push_45deg, SW28(ortho)1 SW_Push_45deg, SW29 SW_Push_45deg, SW29(1.5stagger)1 SW_Push_45deg, SW29(ortho)1 SW_Push_45deg, SW3 SW_Push_45deg, SW30 SW_Push_45deg, SW30(1.5stagger)1 SW_Push_45deg, SW30(ortho)1 SW_Push_45deg, SW31 SW_Push_45deg, SW31(1.5stagger)1 SW_Push_45deg, SW31(ortho)1 SW_Push_45deg, SW32 SW_Push_45deg, SW32(1.5stagger)1 SW_Push_45deg, SW32(ortho)1 SW_Push_45deg, SW33 SW_Push_45deg, SW33(1.5stagger)1 SW_Push_45deg, SW33(ortho)1 SW_Push_45deg, SW34 SW_Push_45deg, SW34(1.5stagger)1 SW_Push_45deg, SW34(ortho)1 SW_Push_45deg, SW35 SW_Push_45deg, SW35(1.5stagger)1 SW_Push_45deg, SW35(ortho)1 SW_Push_45deg, SW36 SW_Push_45deg, SW36(1.5stagger)1 SW_Push_45deg, SW36(ortho)1 SW_Push_45deg, SW37 SW_Push_45deg, SW37(1.5stagger)1 SW_Push_45deg, SW37(ortho)1 SW_Push_45deg, SW38(1.25)1 SW_Push_45deg, SW38(1.5)1 SW_Push_45deg, SW38(ortho)1 SW_Push_45deg, SW39 SW_Push_45deg, SW39(1.5)1 SW_Push_45deg, SW4 SW_Push_45deg, SW40 SW_Push_45deg, SW40(3)1 SW_Push_45deg, SW41 SW_Push_45deg, SW41(1.5)1 SW_Push_45deg, SW42(1.25)1 SW_Push_45deg, SW42(1.5)1 SW_Push_45deg, SW42(3)1 SW_Push_45deg, SW43(1.75)1 SW_Push_45deg, SW43(2)1 SW_Push_45deg, SW44(3)1 SW_Push_45deg, SW44(6)1 SW_Push_45deg, SW45(1.75)1 SW_Push_45deg, SW45(2)1 SW_Push_45deg, SW46(1.25)1 SW_Push_45deg, SW46(1.5)1 SW_Push_45deg, SW46(3)1 SW_Push_45deg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

Commit message: calvin's work
Parts:
- added SW_rotary2: RotaryEncoder_Switch, Keebio-Parts:RotaryEncoder_EC11-no-legs, F.Cu at (261.9, 58.7)
- added SW_rotary3: RotaryEncoder_Switch, Keebio-Parts:RotaryEncoder_EC11-no-legs, F.Cu at (147.6, 58.7)
- added SW_rotary4: RotaryEncoder_Switch, Keebio-Parts:RotaryEncoder_EC11-no-legs, F.Cu at (147.6, 77.8)
- added SW_rotary5: RotaryEncoder_Switch, Keebio-Parts:RotaryEncoder_EC11-no-legs, F.Cu at (100.0, 120.7)
- added SW_rotary6: RotaryEncoder_Switch, Keebio-Parts:RotaryEncoder_EC11-no-legs, F.Cu at (195.3, 120.7)
- C1, C10, C2, C3, C4, C5, C6, C7, C8, C9, D1, D10, D11, D12, D13, D14, D15, D16, D17, D18, D19, D2, D20, D21, D22, D23, D24, D25, D26, D27, D28, D29, D3, D30, D31, D32, D33, D34, D35, D36, D37, D38, D39, D4, D40, D41, D42, D43, D44, D45, D46, D47, D48, D49, D5, D6, D7, D8, D9, F1, R1, R2, SW_Push1, SW_Push3, TP1, TP2, TP3, TP4, TP5, U1, U2, UR1, UR2, UR3, UR4, UR5, UR6, UR7, UR8, USB1, X1: moved to B.Cu
- moved SW26(ISO)1 428.5 mm to (259.6, 87.3)
- moved SW48(3)1 426.9 mm to (238.1, 115.9)
- moved SW12(2)1 386.0 mm to (252.4, 58.7)
- moved SW26(2)1 385.5 mm to (252.4, 77.8)
- moved SW47(1.5)1 370.9 mm to (223.8, 115.9)
- moved SW25(1.5)1 357.0 mm to (257.2, 77.8)
- moved SW45(2)1 355.3 mm to (166.7, 120.7)
- moved SW38(1.5)1 354.2 mm to (257.2, 96.8)
- moved SW49(1.5)1 346.4 mm to (252.4, 115.9)
- moved SW48 341.5 mm to (238.1, 115.9)
- moved SW43(2)1 330.4 mm to (128.6, 120.7)
- moved SW37(1.5stagger)1 327.1 mm to (233.4, 96.8)
- moved OL1 322.6 mm to (147.6, 86.0)
- moved SW45(1.75)1 320.1 mm to (164.3, 120.6)
- moved SW46(1.25)1 316.5 mm to (192.9, 120.6)
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Other:
- board text added: "1 rotary"
- board text added: "2 rotaries"
- board text added: "EDGE CUT NEEDS TO BE ALIGNED TO FOOTPRINTS STILL"
- board text added: "indicator leds"
