File: alpha-curISO_rp2040.kicad_pcb (KiCad board)
At the start: 2 copper layers, 248.6 x 81.9 mm, 195 parts, among them J1 SWD, J2 USB_C_Receptacle_USB2.0, SW1 SW_Push_45deg, SW10 SW_Push_45deg, SW11 SW_Push_45deg, SW12 SW_Push_45deg, SW12(2)1 SW_Push_45deg, SW13 SW_Push_45deg, SW14 SW_Push_45deg, SW15 SW_Push_45deg, SW16 SW_Push_45deg, SW17 SW_Push_45deg, SW18 SW_Push_45deg, SW19 SW_Push_45deg, SW2 SW_Push_45deg, SW20 SW_Push_45deg, SW21 SW_Push_45deg, SW22 SW_Push_45deg, SW23 SW_Push_45deg, SW24 SW_Push_45deg, SW24(1.5)1 SW_Push_45deg, SW25 SW_Push_45deg, SW25(1.5)1 SW_Push_45deg, SW26 SW_Push_45deg, SW26(2)1 SW_Push_45deg, SW26(ISO)1 SW_Push_45deg, SW27 SW_Push, SW27(1.25)1 SW_Push_45deg, SW27(1.5)1 SW_Push_45deg, SW27(ortho)1 SW_Push_45deg, SW28 SW_Push_45deg, SW28(1.5stagger)1 SW_Push_45deg, SW28(ortho)1 SW_Push_45deg, SW29 SW_Push_45deg, SW29(1.5stagger)1 SW_Push_45deg, SW29(ortho)1 SW_Push_45deg, SW3 SW_Push_45deg, SW30 SW_Push_45deg, SW30(1.5stagger)1 SW_Push_45deg, SW30(ortho)1 SW_Push_45deg, SW31 SW_Push_45deg, SW31(1.5stagger)1 SW_Push_45deg, SW31(ortho)1 SW_Push_45deg, SW32 SW_Push_45deg, SW32(1.5stagger)1 SW_Push_45deg, SW32(ortho)1 SW_Push_45deg, SW33 SW_Push_45deg, SW33(1.5stagger)1 SW_Push_45deg, SW33(ortho)1 SW_Push_45deg, SW34 SW_Push_45deg, SW34(1.5stagger)1 SW_Push_45deg, SW34(ortho)1 SW_Push_45deg, SW35 SW_Push_45deg, SW35(1.5stagger)1 SW_Push_45deg, SW35(ortho)1 SW_Push_45deg, SW36 SW_Push_45deg, SW36(1.5stagger)1 SW_Push_45deg, SW36(ortho)1 SW_Push_45deg, SW37 SW_Push_45deg, SW37(1.5stagger)1 SW_Push_45deg, SW37(ortho)1 SW_Push_45deg, SW38(1.25)1 SW_Push_45deg, SW38(1.5)1 SW_Push_45deg, SW38(ortho)1 SW_Push_45deg, SW39 SW_Push_45deg, SW39(1.5)1 SW_Push_45deg, SW4 SW_Push_45deg, SW40 SW_Push_45deg, SW40(3)1 SW_Push_45deg, SW41 SW_Push_45deg, SW41(1.5)1 SW_Push_45deg, SW42(1.25)1 SW_Push_45deg, SW42(1.5)1 SW_Push_45deg, SW42(3)1 SW_Push_45deg, SW43(1.75)1 SW_Push_45deg, SW43(2)1 SW_Push_45deg, SW44(3)1 SW_Push_45deg, SW44(6)1 SW_Push_45deg, SW45(1.75)1 SW_Push_45deg, SW45(2)1 SW_Push_45deg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

Commit message: new position
Parts:
- moved C1 74.9 mm to (111.8, 68.3), turned to -135 degrees
- moved Y1 71.2 mm to (109.5, 66.7), turned to 135 degrees
- moved C2 70.8 mm to (111.1, 65.1), turned to 135 degrees
- moved R7 67.4 mm to (108.3, 68.7), turned to 135 degrees
- moved C14 65.8 mm to (106.3, 69.0), turned to 0 degrees
- moved C9 65.2 mm to (106.3, 68.0), turned to 0 degrees
- moved C11 63.4 mm to (101.0, 73.7), turned to -90 degrees
- moved C8 57.9 mm to (96.8, 73.1), turned to -90 degrees
- moved U1 57.2 mm to (100.0, 66.7), turned to -90 degrees
- moved C16 56.4 mm to (95.6, 73.1), turned to -90 degrees
- moved C13 55.1 mm to (101.0, 59.6), turned to 90 degrees
- moved C7 52.5 mm to (93.7, 70.1), turned to 180 degrees
- moved C10 51.7 mm to (93.7, 69.1), turned to 180 degrees
- moved C17 49.2 mm to (95.9, 61.8), turned to 180 degrees
- moved C15 48.5 mm to (93.0, 66.7), turned to 180 degrees
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Routing:
- net /rp2040 components/USB_BOOT: track 0.00 -> 69.0 mm, vias 0 -> 2
- net +3V3: track 0.00 -> 51.6 mm
- net D_N: track 0.00 -> 50.3 mm
- net D_P: track 0.00 -> 49.4 mm
- net CS: track 0.00 -> 30.1 mm
- net SD1: track 0.00 -> 25.2 mm
- net SD2: track 0.00 -> 21.1 mm
- net VBUS: track 0.00 -> 15.1 mm
- net SD0: track 0.00 -> 12.8 mm
- net QSPI_CLK: track 0.00 -> 12.5 mm
- net SD3: track 0.00 -> 12.3 mm
- net D_USB_N: track 0.00 -> 11.0 mm
- net D_USB_P: track 0.00 -> 9.78 mm
- net XTAL_IN: track 0.00 -> 8.06 mm
- net +5V: track 0.00 -> 7.60 mm
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Other:
- board text removed: "What is the USB position?"
