File: rp2040 components.kicad_sch (KiCad schematic)
At the start: 29 parts, among them J1 SWD, J2 USB_C_Receptacle_USB2.0, SW27 SW_Push, U2 W25Q128JVS, U3 XC6206PxxxMR, U4 USBLC6-2SC6, Y1 12MHz

Commit message: galvy edits - start routing testing
Parts:
- removed J2: USB_C_Receptacle_USB2.0, Connector_USB:USB_C_Receptacle_HRO_TYPE-C-31-M-12, symbol Connector:USB_C_Receptacle_USB2.0
- added USB1: HRO-TYPE-C-31-M-12, Type-C:HRO-TYPE-C-31-M-12-HandSoldering, symbol Type-C:HRO-TYPE-C-31-M-12
Connections:
- net CC1: now also USB1.4 (CC1)
- net CC2: now also USB1.10 (CC2)
- net D_USB_N: now also USB1.5 (DN2), USB1.7 (DN1)
- net D_USB_P: now also USB1.6 (DP1), USB1.8 (DP2)
- net GND: now also USB1.12 (GND), USB1.13 (SHIELD)
- net VBUS: now also USB1.11 (VBUS), USB1.2 (VBUS)

Commit message: corrected schematic component value
Parts:
- C7: value 1nF -> 1uF
Changed lines of the file:
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@@
       (effects (font (size 1.27 1.27)) (justify left))
     )
-    (property "Value" "1nF" (id 1) (at 207.137 83.566 0)
+    (property "Value" "1uF" (id 1) (at 207.137 83.566 0)
       (effects (font (size 1.27 1.27)) (justify left))
     )

Commit message: routing cleanup, first DRC
added a bunch of errors to DRC, should be fine but good to double check
Connections:
- net GND: now also USB1.1 (GND)
Changed lines of the file:
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@@
     (pin "2")
+  )
+  (symbol (lib_id "power:GND") (at 35.56 31.75 90) (unit 1)
+    (in_bom yes) (on_board yes)
+    (property "Reference" "#PWR?" (id 0) (at 41.91 31.75 0)
+      (effects (font (size 1.27 1.27)) hide)
+    )
+    (property "Value" "GND" (id 1) (at 40.64 31.623 0))
+    (property "Footprint" "" (id 2) (at 35.56 31.75 0)
+      (effects (font (size 1.27 1.27)) hide)
+    )
+    (property "Datasheet" "" (id 3) (at 35.56 31.75 0)
+      (effects (font (size 1.27 1.27)) hide)
+    )
+    (pin "1")
   )
   (symbol (lib_id "Device:C_Small") (at 127.762 33.655 90) (unit 1)
