File: Project/plate/plate.kicad_pcb (KiCad board)
At the start: 2 copper layers, 264.5 x 84.3 mm, 16 parts, among them SW27(1.25)1 SW_Push_45deg, SW28 SW_Push_45deg, SW29 SW_Push_45deg, SW30 SW_Push_45deg, SW31 SW_Push_45deg, SW32 SW_Push_45deg, SW33 SW_Push_45deg, SW34 SW_Push_45deg, SW35 SW_Push_45deg, SW36 SW_Push_45deg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

Commit message: fresh production files
Parts:
- removed SW27(1.25)1, SW38(1.25)1: SW_Push_45deg, MX_Only:MXOnly-1.25U-NoLED
- removed SW28, SW29, SW30, SW31, SW32, SW33, SW34, SW35, SW36, SW37: SW_Push_45deg, MX_Only:MXOnly-1U-NoLED
